File: pcb/cheating-calc.kicad_pcb (KiCad board)
At the start: 2 copper layers, 72 x 22 mm, 8 parts, among them J1 Conn_01x04, Q1 MMBF170, Q2 MMBF170, U1 MOUDLE-SEEEDUINO-XIAO-ESP32C3

Commit message: Update cheating-calc.kicad_pcb GXLDVERT 2AM
Other:
- board text added: "TI-32 v0.1 2AM GxldVert 2024"
- board text removed: "TI-32 v0.1 ChromaLock 2024"
Changed lines of the file:
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@@
     )
   )
-  (gr_text "TI-32 v0.1\nChromaLock\n2024" (at 86.487 61.087) (layer "F.SilkS")
+  (gr_text "TI-32 v0.1\n2AM GxldVert\n2024" (at 86.487 61.087) (layer "F.SilkS")
     (effects (font (face "Joystix Monospace") (size 1.7 1.7) (thickness 0.2) bold) (justify left bottom))
     (render_cache "TI-32 v0.1\nChromaLock\n2024" 0
